File: hardware/Air858.sch (EAGLE design)
At the start: 54 parts, among them IC1 ATMEGA168, IC2 MAX31855, IC3 LD117, Q1 TSM3404, SW1 EC12E_SW, T1 BTA16, X1 CSTCR6M00G53Z

Commit message: fix schematic issues and update board
Parts:
- added 0V, I, V, VCC, ZX: PTR1B1,27, testpad:PTR1B1,27
- R2: device rcl:R-EU_R0603 -> rcl:R-EU_M1206
Connections:
- net +24V: no longer R5.2
- net +3V3: now also VCC.TP
- net 10V_AC1: now also TX1-4.S; no longer TX1-1.S
- net 25V_AC1: now also TX1-2.S; no longer TX1-3.S
- net 25V_AC2: now also TX1-1.S; no longer TX1-4.S
- net FAN-: now also R5.2
- net FAN_SENSE_I: now also I.TP
- net FAN_SENSE_V: now also V.TP
- net GND: now also 0V.TP, TX1-3.S; no longer TX1-2.S
- net SW2: now also IC1.ADC2/ANALOG_2/PC2; no longer IC1.ADC7
- net ZEROX: now also ZX.TP
Other:
- moved on the sheet: R5, TX1-1, TX1-2, TX1-3, TX1-4
Changed lines of the file:
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@@
 <part name="Q1" library="adafruit" deviceset="MOSFET-N" device="REFLOW" value="TSM3404"/>
 <part name="D9" library="diode" deviceset="DIODE-" device="DO-214AC"/>
-<part name="R2" library="rcl" deviceset="R-EU_" device="R0603" value="10R"/>
+<part name="R2" library="rcl" deviceset="R-EU_" device="M1206" value="10R"/>
 <part name="GND2" library="supply1" deviceset="GND" device=""/>
 <part name="C7" library="rcl" deviceset="C-EU" device="C0603K" value="100n"/>
@@
 <part name="X1" library="murata-filter" deviceset="CSTCR" device="" technology="6M00G53Z"/>
 <part name="R1" library="rcl" deviceset="R-EU_" device="R0603" value="47k"/>
+<part name="V" library="testpad" deviceset="PTR1" device="B1,27"/>
+<part name="I" library="testpad" deviceset="PTR1" device="B1,27"/>
+<part name="VCC" library="testpad" deviceset="PTR1" device="B1,27"/>
+<part name="ZX" library="testpad" deviceset="PTR1" device="B1,27"/>
+<part name="0V" library="testpad" deviceset="PTR1" device="B1,27"/>
 </parts>
 <sheets>
 <sheet>
 <plain>
-<text x="182.88" y="-45.72" size="1.27" layer="97">max. fan current ~380mA</text>
+<text x="154.94" y="-45.72" size="1.27" layer="97">max. fan current ~380mA</text>
 <text x="132.08" y="-5.08" size="1.27" layer="97">actually ~36V</text>
 </plain>
@@
 </instance>
 <instance part="OK1" gate="-1" x="165.1" y="48.26"/>
-<instance part="TX1" gate="-1" x="-30.48" y="55.88" smashed="yes" rot="MR0">
-<attribute name="NAME" x="-33.02" y="55.118" size="1.524" layer="95" rot="MR0"/>
-</instance>
-<instance part="TX1" gate="-2" x="-30.48" y="43.18" rot="MR0"/>
-<instance part="TX1" gate="-3" x="109.22" y="-17.78" rot="MR0"/>
-<instance part="TX1" gate="-4" x="109.22" y="-20.32" rot="MR0"/>
+<instance part="TX1" gate="-1" x="104.14" y="-22.86" smashed="yes" rot="MR0">
+<attribute name="NAME" x="101.6" y="-23.622" size="1.524" layer="95" rot="MR0"/>
+</instance>
+<instance part="TX1" gate="-2" x="104.14" y="-15.24" rot="MR0"/>
+<instance part="TX1" gate="-3" x="-30.48" y="50.8" rot="MR0"/>
+<instance part="TX1" gate="-4" x="-30.48" y="55.88" rot="MR0"/>
 <instance part="C1X" gate="G$1" x="200.66" y="35.56" smashed="yes" rot="R180">
 <attribute name="NAME" x="197.866" y="36.957" size="1.778" layer="95" rot="R180"/>
@@
 <instance part="GND6" gate="1" x="66.04" y="2.54" smashed="yes"/>
 <instance part="R4" gate="G$1" x="167.64" y="-25.4" rot="R90"/>
-<instance part="R5" gate="G$1" x="198.12" y="-5.08" rot="R90"/>
+<instance part="R5" gate="G$1" x="193.04" y="-5.08" rot="R180"/>
 <instance part="R6" gate="G$1" x="198.12" y="-25.4" rot="R90"/>
 <instance part="R7" gate="G$1" x="215.9" y="-25.4" rot="R90"/>
 <instance part="C12" gate="G$1" x="205.74" y="-22.86"/>
-<instance part="GND8" gate="1" x="-20.32" y="38.1"/>
+<instance part="GND8" gate="1" x="-25.4" y="38.1"/>
 <instance part="FAN" gate="-1" x="165.1" y="0" smashed="yes" rot="R180">
 <attribute name="NAME" x="162.56" y="0.762" size="1.524" layer="95" rot="R180"/>
@@
 <instance part="X1" gate="G$1" x="55.88" y="38.1"/>
 <instance part="R1" gate="G$1" x="-20.32" y="71.12"/>
+<instance part="V" gate="G$1" x="218.44" y="-35.56" rot="R90"/>
+<instance part="I" gate="G$1" x="195.58" y="-35.56" rot="R90"/>
+<instance part="VCC" gate="G$1" x="20.32" y="55.88" rot="R90"/>
+<instance part="ZX" gate="G$1" x="-7.62" y="71.12" rot="R90"/>
+<instance part="0V" gate="G$1" x="53.34" y="22.86" rot="R270"/>
 </instances>
 <busses>
@@
 <pinref part="D1" gate="G$1" pin="A"/>
 <pinref part="D3" gate="G$1" pin="C"/>
-<wire x1="119.38" y1="-15.24" x2="119.38" y2="-17.78" width="0.1524" layer="91"/>
-<wire x1="119.38" y1="-17.78" x2="119.38" y2="-22.86" width="0.1524" layer="91"/>
-<wire x1="119.38" y1="-17.78" x2="111.76" y2="-17.78" width="0.1524" layer="91"/>
-<junction x="119.38" y="-17.78"/>
-<label x="106.68" y="-15.24" size="1.27" layer="95"/>
-<pinref part="TX1" gate="-3" pin="S"/>
+<wire x1="119.38" y1="-15.24" x2="119.38" y2="-22.86" width="0.1524" layer="91"/>
+<wire x1="119.38" y1="-15.24" x2="106.68" y2="-15.24" width="0.1524" layer="91"/>
+<junction x="119.38" y="-15.24"/>
+<label x="107.696" y="-17.272" size="1.27" layer="95"/>
+<pinref part="TX1" gate="-2" pin="S"/>
 </segment>
 </net>
@@
 <pinref part="D2" gate="G$1" pin="A"/>
 <pinref part="D4" gate="G$1" pin="C"/>
-<wire x1="129.54" y1="-15.24" x2="129.54" y2="-20.32" width="0.1524" layer="91"/>
-<wire x1="129.54" y1="-20.32" x2="129.54" y2="-22.86" width="0.1524" layer="91"/>
-<wire x1="129.54" y1="-20.32" x2="111.76" y2="-20.32" width="0.1524" layer="91"/>
-<junction x="129.54" y="-20.32"/>
-<label x="106.68" y="-22.86" size="1.27" layer="95"/>
-<pinref part="TX1" gate="-4" pin="S"/>
+<wire x1="129.54" y1="-15.24" x2="129.54" y2="-22.86" width="0.1524" layer="91"/>
+<wire x1="129.54" y1="-22.86" x2="106.68" y2="-22.86" width="0.1524" layer="91"/>
+<junction x="129.54" y="-22.86"/>
+<label x="107.442" y="-21.844" size="1.27" layer="95"/>
+<pinref part="TX1" gate="-1" pin="S"/>
 </segment>
 </net>
@@
 <wire x1="55.88" y1="30.48" x2="55.88" y2="22.86" width="0.1524" layer="91"/>
 <wire x1="55.88" y1="22.86" x2="66.04" y2="22.86" width="0.1524" layer="91"/>
-</segment>
-<segment>
-<wire x1="-27.94" y1="43.18" x2="-20.32" y2="43.18" width="0.1524" layer="91"/>
-<wire x1="-20.32" y1="43.18" x2="-20.32" y2="40.64" width="0.1524" layer="91"/>
+<pinref part="0V" gate="G$1" pin="TP"/>
+<junction x="55.88" y="22.86"/>
+</segment>
+<segment>
+<wire x1="-27.94" y1="50.8" x2="-25.4" y2="50.8" width="0.1524" layer="91"/>
+<wire x1="-25.4" y1="50.8" x2="-25.4" y2="40.64" width="0.1524" layer="91"/>
 <pinref part="GND8" gate="1" pin="GND"/>
-<pinref part="TX1" gate="-2" pin="S"/>
+<pinref part="TX1" gate="-3" pin="S"/>
 </segment>
 <segment>
@@
 <pinref part="P+3" gate="1" pin="+24V"/>
 <wire x1="177.8" y1="5.08" x2="177.8" y2="0" width="0.1524" layer="91"/>
-<wire x1="177.8" y1="0" x2="182.88" y2="0" width="0.1524" layer="91"/>
 <junction x="177.8" y="0"/>
 <label x="168.402" y="1.016" size="1.27" layer="95"/>
 <wire x1="177.8" y1="0" x2="167.64" y2="0" width="0.1524" layer="91"/>
 <pinref part="FAN" gate="-1" pin="S"/>
-</segment>
-<segment>
-<pinref part="R5" gate="G$1" pin="2"/>
-<wire x1="198.12" y1="0" x2="182.88" y2="0" width="0.1524" layer="91"/>
 </segment>
 </net>
@@
 <segment>
 <pinref part="D5" gate="G$1" pin="A"/>
-<pinref part="TX1" gate="-1" pin="S"/>
 <wire x1="-27.94" y1="55.88" x2="-25.4" y2="55.88" width="0.1524" layer="91"/>
 <pinref part="R1" gate="G$1" pin="1"/>
 <wire x1="-25.4" y1="55.88" x2="-25.4" y2="71.12" width="0.1524" layer="91"/>
 <junction x="-25.4" y="55.88"/>
+<pinref part="TX1" gate="-4" pin="S"/>
 </segment>
 </net>
@@
 <pinref part="IC1" gate="G$1" pin="PC6/RESET"/>
 <wire x1="68.58" y1="68.58" x2="60.96" y2="68.58" width="0.1524" layer="91"/>
-<label x="50.8" y="68.58" size="1.27" layer="95"/>
+<label x="58.42" y="69.596" size="1.27" layer="95"/>
 </segment>
 </net>
@@
 <label x="167.64" y="-7.62" size="1.27" layer="95"/>
 <pinref part="FAN" gate="-2" pin="S"/>
+<pinref part="R5" gate="G$1" pin="2"/>
+<wire x1="177.8" y1="-5.08" x2="187.96" y2="-5.08" width="0.1524" layer="91"/>
 </segment>
 </net>
@@
 <segment>
 <pinref part="R7" gate="G$1" pin="1"/>
-<wire x1="215.9" y1="-30.48" x2="215.9" y2="-38.1" width="0.1524" layer="91"/>
-<label x="222.758" y="-39.116" size="1.27" layer="95" rot="R180"/>
+<wire x1="215.9" y1="-30.48" x2="215.9" y2="-35.56" width="0.1524" layer="91"/>
+<label x="222.758" y="-44.196" size="1.27" layer="95" rot="R180"/>
+<pinref part="V" gate="G$1" pin="TP"/>
+<wire x1="215.9" y1="-35.56" x2="215.9" y2="-43.18" width="0.1524" layer="91"/>
+<junction x="215.9" y="-35.56"/>
 </segment>
 <segment>
@@
 <wire x1="185.42" y1="-20.32" x2="185.42" y2="-17.78" width="0.1524" layer="91"/>
 <wire x1="185.42" y1="-17.78" x2="193.04" y2="-17.78" width="0.1524" layer="91"/>
-<label x="199.39" y="-39.878" size="1.27" layer="95" rot="R180"/>
-<wire x1="193.04" y1="-17.78" x2="193.04" y2="-38.1" width="0.1524" layer="91"/>
+<label x="199.39" y="-44.958" size="1.27" layer="95" rot="R180"/>
+<wire x1="193.04" y1="-17.78" x2="193.04" y2="-35.56" width="0.1524" layer="91"/>
 <pinref part="Q1" gate="G$1" pin="S"/>
 <pinref part="R2" gate="G$1" pin="2"/>
+<wire x1="193.04" y1="-35.56" x2="193.04" y2="-43.18" width="0.1524" layer="91"/>
 <wire x1="177.8" y1="-20.32" x2="177.8" y2="-17.78" width="0.1524" layer="91"/>
 <wire x1="177.8" y1="-17.78" x2="185.42" y2="-17.78" width="0.1524" layer="91"/>
 <junction x="185.42" y="-17.78"/>
 <junction x="177.8" y="-17.78"/>
+<pinref part="I" gate="G$1" pin="TP"/>
+<junction x="193.04" y="-35.56"/>
 </segment>
 <segment>
@@
 <pinref part="R6" gate="G$1" pin="2"/>
 <wire x1="198.12" y1="-20.32" x2="198.12" y2="-17.78" width="0.1524" layer="91"/>
-<wire x1="198.12" y1="-17.78" x2="198.12" y2="-10.16" width="0.1524" layer="91"/>
+<wire x1="198.12" y1="-17.78" x2="198.12" y2="-5.08" width="0.1524" layer="91"/>
 <wire x1="205.74" y1="-17.78" x2="198.12" y2="-17.78" width="0.1524" layer="91"/>
 <junction x="198.12" y="-17.78"/>
@@
 <label x="-10.16" y="73.66" size="1.27" layer="95"/>
 <pinref part="R1" gate="G$1" pin="2"/>
+<pinref part="ZX" gate="G$1" pin="TP"/>
 </segment>
 <segment>
@@
 <wire x1="10.16" y1="63.5" x2="10.16" y2="55.88" width="0.1524" layer="91"/>
 <pinref part="+3V5" gate="G$1" pin="+3V3"/>
+<pinref part="VCC" gate="G$1" pin="TP"/>
 </segment>
 <segment>
@@
 </segment>
 <segment>
-<pinref part="IC1" gate="G$1" pin="ADC7"/>
-<wire x1="129.54" y1="50.8" x2="134.62" y2="50.8" width="0.1524" layer="91"/>
-<label x="134.62" y="50.8" size="1.27" layer="95"/>
-</segment>
-</net>
+<pinref part="IC1" gate="G$1" pin="ADC2/ANALOG_2/PC2"/>
+<wire x1="129.54" y1="63.5" x2="134.62" y2="63.5" width="0.1524" layer="91"/>
+<label x="134.62" y="63.5" size="1.27" layer="95"/>
+</segment>
+</net>

Commit message: rev 1: prototype
Parts:
- C3: device rcl:CPOL-EU153CLV-0810 -> rcl:CPOL-EUSMCE
- C4: device rcl:CPOL-EUB/3528-21W -> rcl:CPOL-EUSMCE
Changed lines of the file:
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@@
 <part name="IC3" library="v-reg" deviceset="LD117A?*" device="S" technology="12TR" value="LD117"/>
 <part name="C2" library="rcl" deviceset="C-EU" device="C0603" value="100~n"/>
-<part name="C3" library="rcl" deviceset="CPOL-EU" device="153CLV-0810" value="220µ"/>
-<part name="C4" library="rcl" deviceset="CPOL-EU" device="B/3528-21W" value="220µ"/>
+<part name="C3" library="rcl" deviceset="CPOL-EU" device="SMCE" value="220µ"/>
+<part name="C4" library="rcl" deviceset="CPOL-EU" device="SMCE" value="220µ"/>
 <part name="T1" library="triac" deviceset="TIC206" device="" technology="D" value="BTA16"/>
 <part name="OK1" library="optocoupler" deviceset="MOC30*" device="" technology="41M"/>
