File: hardware/Air858.brd (EAGLE design)
At the start: 75 x 93 mm, 60 parts, among them IC1 ATMEGA168, IC2 MAX31855, IC3 LD117, Q1 TSM3404, SW1 EC12E_SW, T1 BTA16, X1 CSTCR6M00G53Z

Commit message: changed zero crossing detection based on AVR182
Parts:
- removed OK2: H11A1M, optocoupler:DIL06
- removed R101, R102: 47k, rcl:M1206
- added R1: 47k, rcl:R0603
- moved R104 11.9 mm to (19.1, 76.8), turned to 90 degrees
- moved R3 11.8 mm to (18.7, 47.9)
- moved OK1 10.2 mm to (16.5, 55.2)
- moved R103 10.2 mm to (14.0, 64.1)
- moved R105 10.2 mm to (19.1, 64.1)
- moved C1X 5.12 mm to (22.9, 77.5), turned to 270 degrees
- moved T1 4.07 mm to (6.99, 69.2), turned to 270 degrees
- moved U$5 3.17 mm to (7.62, 69.2), turned to 90 degrees
- moved IC2 0.64 mm to (38.7, 13.3)
- moved C9 0.64 mm to (38.7, 8.26)
- moved TC 0.64 mm to (37.5, 3.81)
- moved C8 0.63 mm to (42.2, 12.7)
Connections:
- removed net N$2: OK2.1, R101.2
- removed net N$7: OK2.2, R102.2
- net 10V_AC1: now also R1.1
- net GND: no longer OK2.4
- net MAINS_L: no longer R101.1
- net MAINS_N: no longer R102.1
- net ZEROX: now also R1.2; no longer OK2.5
Routing:
- net ZEROX: track 21.5 -> 77.2 mm, vias 0 -> 2
- net MAINS_L: track 72.6 -> 51.5 mm
- net HEATER_DRIVE: track 30.0 -> 42.4 mm, vias 0 -> 1
- net HEATER: track 32.1 -> 20.6 mm
- net +3V3: track 190.9 -> 180.4 mm
- net 10V_AC1: track 24.9 -> 31.3 mm
- net N$8: track 19.7 -> 24.0 mm
- net N$2: track 3.94 -> 0.00 mm
- net N$7: track 3.68 -> 0.00 mm
- net N$9: track 1.91 -> 4.60 mm
- net MAINS_N: track 65.6 -> 66.8 mm, vias 0 -> 1
- net SS: track 56.9 -> 56.2 mm
- net REED: track 55.4 -> 54.8 mm
- net SCK: track 78.4 -> 77.8 mm
- net MISO: track 67.9 -> 67.3 mm
Other:
- outline, holes or cut-outs redrawn

Commit message: fix schematic issues and update board
Parts:
- added 0V, I, V, VCC, ZX: PTR1B1,27, testpad:B1,27
- R2: device rcl:R0603 -> rcl:M1206
- moved LA1 1.91 mm to (44.1, 58.4)
- moved C14 1.85 mm to (44.1, 61.9)
- moved R5 0.95 mm to (69.2, 20.0), turned to 180 degrees
- moved C12 0.64 mm to (69.2, 24.4)
- moved R6 0.64 mm to (69.2, 22.2)
- moved R7 0.64 mm to (69.2, 26.7)
- moved D9 0.63 mm to (69.2, 8.26)
- moved R2 0.63 mm to (64.1, 19.7)
- moved C7 0.32 mm to (62.2, 19.1)
Connections:
- net +24V: no longer R5.2
- net +3V3: now also VCC.TP
- net 10V_AC1: now also TX1.4; no longer TX1.1
- net 25V_AC1: now also TX1.2; no longer TX1.3
- net 25V_AC2: now also TX1.1; no longer TX1.4
- net FAN-: now also R5.2
- net FAN_SENSE_I: now also I.TP
- net FAN_SENSE_V: now also V.TP
- net GND: now also 0V.TP, TX1.3; no longer TX1.2
- net SW2: now also IC1.25; no longer IC1.22
- net ZEROX: now also ZX.TP
Routing:
- net 10V_AC1: track 31.3 -> 14.2 mm, vias 1 -> 0
- net 25V_AC2: track 32.1 -> 18.8 mm, vias 0 -> 1
- net FAN-: track 11.3 -> 19.2 mm
- net +3V3: track 180.4 -> 183.0 mm
- net SW2: track 48.4 -> 46.6 mm
- net AVCC: track 7.11 -> 5.62 mm
- net +24V: track 71.9 -> 70.4 mm
- net N$1: track 8.08 -> 6.69 mm
- net ZEROX: track 77.2 -> 78.5 mm
- net MAINS_L: track 51.5 -> 52.1 mm
- net FAN: track 52.1 -> 52.7 mm
- net FAN_SENSE_I: track 65.2 -> 64.6 mm

Commit message: rev 1: prototype
Parts:
- C3: device rcl:153CLV-0810 -> rcl:SMC_E
- C4: device rcl:B/3528-21W -> rcl:SMC_E
- moved 0V 17.4 mm to (48.9, 61.6)
- moved VCC 14.8 mm to (48.9, 58.4)
- moved C5 8.91 mm to (64.1, 71.1), turned to 90 degrees
- moved D6 3.70 mm to (56.5, 59.7), turned to 270 degrees
- moved C4 3.17 mm to (61.0, 58.4), turned to 270 degrees
- moved C8 2.13 mm to (43.2, 10.8), turned to 0 degrees
- moved C2 1.91 mm to (55.2, 66.0), turned to 90 degrees
- moved C3 1.91 mm to (56.5, 75.2), turned to 180 degrees
Routing:
- net +3V3: track 183.0 -> 164.1 mm, vias 5 -> 3
- net N$4: track 28.0 -> 23.9 mm
- net SS: track 56.2 -> 56.7 mm

Commit message: add oshw logo
Parts:
- added U$6: (no value), adafruit:OSHWLOGO_TOP_0.2
Changed lines of the file:
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@@
 <attribute name="VALUE" x="48.26" y="60.833" size="0.0254" layer="27"/>
 </element>
+<element name="U$6" library="adafruit" package="OSHWLOGO_TOP_0.2" value="" x="28.575" y="26.67"/>
 </elements>
 <signals>
